Commit message: feat: Update URDF Sirius and change param laser filter

File: msd700_visual/urdf/msd700_sirius.urdf.xacro (robot description, xacro)
@@ -213,30 +213,4 @@
     <origin xyz="-0.06 0 0.15" rpy="0 0 0"/>
   </joint>
-  <!-- Sensor Ultrasonik -->
-  <link name="ultrasonic_sensor_link">
-    <visual>
-      <origin xyz="0 0 0" rpy="1.57 0 0"/>
-      <geometry>
-      <cylinder length="0.05" radius="0.01" />
-      </geometry>
-      <material name="dark"/>
-    </visual>
-    <collision>
-      <origin xyz="0 0 0" rpy="0 0 0"/>
-      <geometry>
-        <cylinder length="0.05" radius="0.01" />
-      </geometry>
-    </collision>
-    <inertial>
-      <mass value="0.01" />
-      <origin xyz="0 0 0" rpy="0 0 0" />
-      <inertia ixx="1e-5" iyy="1e-5" izz="1e-5" ixy="0" ixz="0" iyz="0" />
-    </inertial>
-  </link>
-  <joint name="ultrasonic_sensor_joint" type="fixed">
-    <parent link="base_link" />
-    <child link="ultrasonic_sensor_link" />
-    <origin xyz="-0.2 0 0.05" rpy="0 0 3.14159" />
-  </joint>
   <joint name="camera_joint" type="fixed">
     <origin xyz="0.064 -0.065 0.094" rpy="0 0 0"/>
